File: keyboard.kicad_sch (KiCad schematic)
At the start: 184 parts, among them J1 USB_mini_micro_B, K1 KEYSW, K10 KEYSW, K11 KEYSW, K12 KEYSW, K13 KEYSW, K14 KEYSW, K15 KEYSW, K16 KEYSW, K17 KEYSW, K18 KEYSW, K19 KEYSW, K2 KEYSW, K20 KEYSW, K21 KEYSW, K22 KEYSW, K23 KEYSW, K24 KEYSW, K25 KEYSW, K26 KEYSW, K27 KEYSW, K28 KEYSW, K29 KEYSW, K3 KEYSW, K30 KEYSW, K31 KEYSW, K32 KEYSW, K33 KEYSW, K34 KEYSW, K35 KEYSW, K36 KEYSW, K37 KEYSW, K38 KEYSW, K39 KEYSW, K4 KEYSW, K40 KEYSW, K41 KEYSW, K42 KEYSW, K43 KEYSW, K44 KEYSW, K45 KEYSW, K46 KEYSW, K47 KEYSW, K48 KEYSW, K49 KEYSW, K5 KEYSW, K50 KEYSW, K51 KEYSW, K52 KEYSW, K53 KEYSW, K54 KEYSW, K55 KEYSW, K56 KEYSW, K57 KEYSW, K58 KEYSW, K59 KEYSW, K6 KEYSW, K60 KEYSW, K61 KEYSW, K62 KEYSW, K63 KEYSW, K64 KEYSW, K65 KEYSW, K66 KEYSW, K67 KEYSW, K68 KEYSW, K69 KEYSW, K7 KEYSW, K70 KEYSW, K71 KEYSW, K72 KEYSW, K73 KEYSW, K74 KEYSW, K75 KEYSW, K76 KEYSW, K78 KEYSW, K8 KEYSW, K81 KEYSW, K85 KEYSW, K86 KEYSW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

Commit message: splitted the keyboard, added OLED and changed microcontroller, TODO: add footprints for microcontrollers, keys and diodes
Parts:
- removed C1, C2: 22p, symbol Device:C_Small
- removed C3, C4, C5, C6: 0.1u, symbol Device:C_Small
- removed C7: 4.7u, symbol Device:C_Small
- removed C8: 1u, symbol Device:C_Small
- removed D85, D86, D87, D88, D89, D90: D, symbol Device:D
- removed J1: USB_mini_micro_B, symbol keyboard_parts:USB_mini_micro_B
- removed K85, K86, K87, K88, K89, K90: KEYSW, symbol keyboard_parts:KEYSW
- removed R1, R2: 10k, symbol Device:R
- removed R3, R4: 22, symbol Device:R
- removed SW1: SW_PUSH, symbol keyboard_parts:SW_PUSH
- removed U1: ATMEGA32U4, symbol keyboard_parts:ATMEGA32U4
- removed X1: XTAL_GND, symbol keyboard_parts:XTAL_GND
- added D77, D79, D80: 1n4148, symbol Device:D
- added K77, K79, K80: KEYSW, symbol keyboard_parts:KEYSW
- added U1, U2: nRF52840_Featherwing, symbol nrf52840_featherwing:nRF52840_Featherwing
- added U3, U4: ~, 1_my_custom_footprint_library:SSD1306-0.91-OLED-4pin-128x32, symbol 1_my_custom_symbol_library:OLED_4pin_0.91_128*32
- D1, D10, D11, D12, D13, D14, D15, D16, D17, D18, D19, D2, D20, D21, D22, D23, D24, D25, D26, D27, D28, D29, D3, D30, D31, D32, D33, D34, D35, D36, D37, D38, D39, D4, D40, D41, D42, D43, D44, D45, D46, D47, D48, D49, D5, D50, D51, D52, D53, D54, D55, D56, D57, D58, D59, D6, D60, D61, D62, D63, D64, D65, D66, D67, D68, D69, D7, D70, D71, D72, D73, D74, D75, D76, D78, D8, D9: value D -> 1n4148
- D81: value D -> 1N4148; footprint (none) -> Diode_THT:D_DO-35_SOD27_P7.62mm_Horizontal
Connections:
- net at D68.1 (K), D69.1 (K), D70.1 (K)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: now also U2.20 (GPIO6); no longer D60.1 (K), D62.1 (K), D63.1 (K), D64.1 (K), D65.1 (K), D66.1 (K), D67.1 (K)
- net at D75.1 (K), D76.1 (K), D78.1 (K): now also D77.1 (K), D79.1 (K), D80.1 (K), U2.19 (GPIO5); no longer D81.1 (K)
- net at D53.1 (K), D54.1 (K), D55.1 (K)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: now also D60.1 (K), U2.22 (GPIO10); no longer D47.1 (K), D48.1 (K), D49.1 (K), D50.1 (K), D51.1 (K), D52.1 (K), D61.1 (K)
- net at D38.1 (K), D39.1 (K), D40.1 (K)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: now also U2.25 (GPIO13); no longer D32.1 (K), D33.1 (K), D34.1 (K), D35.1 (K), D36.1 (K), D37.1 (K), D46.1 (K)
- net at D46.2 (A), K46.2: now also U2.24 (GPIO12)
- net at K44.1, K59.1: now also K52.1, K67.1, K74.1, U2.8 (GPIOA3); no longer K14.1, K73.1
- net at K43.1, K58.1: now also K51.1, K66.1, K73.1, K80.1, U2.9 (GPIOA4); no longer K13.1, K29.1
- new net: D80.2 (A), K80.2
- new net: D46.1 (K), D47.1 (K), D48.1 (K), D49.1 (K), D50.1 (K), D51.1 (K), D52.1 (K), U2.23 (GPIO11)
- new net: K38.1, K46.1, K53.1, K61.1, K68.1, K75.1
- new net: D10.1 (K), D11.1 (K), D12.1 (K), D13.1 (K), D14.1 (K), D8.1 (K), D9.1 (K), U1.24 (GPIO12)
- new net: K16.1, K2.1, K22.1, K28.1, K34.1, K9.1, U1.13 (GPIOMISO)
- new net: K41.1, K49.1, K56.1, K64.1, K71.1, K78.1, U2.11 (GPIOSCK)
- new net: K13.1, K20.1, K26.1, K32.1, K6.1, K81.1, U1.9 (GPIOA4)
- new net: D21.1 (K), D22.1 (K), D23.1 (K), D24.1 (K), D25.1 (K), D26.1 (K), U1.22 (GPIO10)
- new net: K39.1, K47.1, K54.1, K62.1, K69.1, K76.1, U2.13 (GPIOMISO)
- new net: D61.1 (K), D62.1 (K), D63.1 (K), D64.1 (K), D65.1 (K), D66.1 (K), D67.1 (K), U2.21 (GPIO9)
- new net: D1.1 (K), D2.1 (K), D3.1 (K), D4.1 (K), D5.1 (K), D6.1 (K), D7.1 (K), U1.25 (GPIO13)
- new net: K11.1, K18.1, K24.1, K30.1, K36.1, K4.1, U1.11 (GPIOSCK)
- new net: D15.1 (K), D16.1 (K), D17.1 (K), D18.1 (K), D19.1 (K), D20.1 (K), U1.23 (GPIO11)
- new net: K40.1, K48.1, K55.1, K63.1, K70.1, K77.1, U2.12 (GPIOMOSI)
- new net: D27.1 (K), D28.1 (K), D29.1 (K), D30.1 (K), D31.1 (K), D32.1 (K), U1.21 (GPIO9)
- new net: K45.1, K60.1, U2.7 (GPIOA2)
- new net: K1.1, K15.1, K21.1, K27.1, K33.1, K8.1, U1.14 (GPIORX)
- new net: K12.1, K19.1, K25.1, K31.1, K37.1, K5.1, U1.10 (GPIOA5)
- new net: K10.1, K17.1, K23.1, K29.1, K3.1, K35.1, U1.12 (GPIOMOSI)
- new net: K42.1, K50.1, K57.1, K65.1, K72.1, K79.1, U2.10 (GPIOA5)
- new net: D33.1 (K), D34.1 (K), D35.1 (K), D36.1 (K), D37.1 (K), D81.1 (K), U1.20 (GPIO6)
- new net: U1.17 (SDA), U4. (VCC)
- new net: U1.18 (SCL), U4. (VCC)
- new net: U1.2 (3V), U4. (VCC)
- new net: U1.4 (GND), U4. (VCC)
- new net: K14.1, K7.1, U1.8 (GPIOA3)
- new net: U2.17 (SDA), U3. (VCC)
- new net: U2.18 (SCL), U3. (VCC)
- new net: U2.2 (3V), U3. (VCC)
- new net: U2.4 (GND), U3. (VCC)
- new net: D77.2 (A), K77.2
- new net: D79.2 (A), K79.2
Other:
- moved on the sheet: D1, D2, D3, D4, D5, D6, D7, K1, K2, K3, K4, K5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
